File: 880_case.kicad_pcb (KiCad board)
At the start: 2 copper layers, 163 parts, among them CON1 BARREL_JACK, J1 RUN/STOP, J10 RS IN, J11 CP IN, J12 MA IN, J13 CB IN, J14 CY IN, J15 OH IN, J16 CH IN, J17 IN 1, J18 IN 2, J19 IN 3, J2 SYNC24 CLK, J20 IN 4, J21 MULT IN, J22 SUM, J23 JACK_STEREO, J3 ASSIGN 1, J4 ASSIGN 2, J5 BD IN, J6 SD IN, J7 LT IN, J8 MT IN, J9 HT IN, P1 CONN_02X03, P2 CONN_01X02, P3 CONN_02X05, P4 CONN_01X03, Q1 MMBT3904, Q10 MMBT3904, Q11 MMBT3904, Q12 MMBT3904, Q13 MMBT3904, Q14 C945, Q15 A733, Q2 MMBT3904, Q3 MMBT3904, Q4 MMBT3904, Q5 MMBT3904, Q6 MMBT3904, Q7 MMBT3904, Q8 MMBT3904, Q9 MMBT3904, U1 74HC165, U2 74HC165, U3 VX078-500, U4 VX078-500, U5 4558, U6 4558, X1 MIDI OUT, X2 SYNC24

Commit message: more component placement
Parts:
- C1, C10, C4, C5, C6, C7, C8, C9, D1, D17, D2, D3, D4, D5, L1, L2, L3, L4, P2, Q1, R1, R10, R14, R2, R3, R4, R5, R6, U1, U2, U5, U6: moved to B.Cu
- moved P4 228.8 mm to (268.5, 74.5)
- moved J22 225.2 mm to (259.0, 64.0), turned to 90 degrees
- moved J21 219.1 mm to (259.0, 77.0), turned to 90 degrees
- moved J19 209.7 mm to (241.0, 64.0), turned to 90 degrees
- moved J20 203.2 mm to (241.0, 77.0), turned to 90 degrees
- moved U6 199.0 mm to (242.0, 88.0)
- moved J17 194.6 mm to (223.0, 64.0), turned to 90 degrees
- moved U5 191.0 mm to (233.0, 88.0)
- moved J18 187.5 mm to (223.0, 77.0), turned to 90 degrees
- moved J15 180.0 mm to (205.0, 64.0), turned to 90 degrees
- moved J16 172.4 mm to (205.0, 77.0), turned to 90 degrees
- moved J13 166.1 mm to (187.0, 64.0), turned to 90 degrees
- moved J14 157.8 mm to (187.0, 77.0), turned to 90 degrees
- moved J11 153.1 mm to (169.0, 64.0), turned to 90 degrees
- moved J12 144.4 mm to (169.5, 77.0), turned to 90 degrees
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
Commit message: more placement
Parts:
- D10, D11, D12, D6, D7, D8, D9, Q2, Q3, Q4, Q5, Q6, Q7, Q8, R11, R12, R13, R15, R16, R17, R18, R19, R20, R21, R22, R23, R24, R25, R26, R27, R28, R29, R7, R8, R9: moved to B.Cu
- moved R20 148.9 mm to (161.8, 63.0), turned to 270 degrees
- moved D11 147.8 mm to (159.8, 62.8), turned to 270 degrees
- moved R24 146.6 mm to (158.2, 63.0), turned to 90 degrees
- moved Q7 145.5 mm to (160.8, 66.8)
- moved R28 143.4 mm to (158.2, 67.2), turned to 270 degrees
- moved R21 139.5 mm to (161.8, 76.0), turned to 270 degrees
- moved D12 138.2 mm to (159.8, 75.8), turned to 270 degrees
- moved R18 137.6 mm to (143.8, 63.0), turned to 270 degrees
- moved R25 137.0 mm to (158.2, 76.0), turned to 90 degrees
- moved D9 136.6 mm to (141.8, 62.8), turned to 270 degrees
- moved Q8 136.0 mm to (160.8, 80.0)
- moved R22 135.5 mm to (140.2, 63.0), turned to 90 degrees
- moved Q5 134.0 mm to (142.8, 66.8)
- moved R29 133.8 mm to (158.2, 80.5), turned to 270 degrees
- moved R26 132.1 mm to (140.2, 67.2), turned to 270 degrees
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
Commit message: added 3d models for DC jack, VX0-78XX-500 DC-DC converters, and stereo headhpone jack
Parts:
- C11, C12, C13, C14, C15, C16, C17, C18, C2, C23, C3, D13, D14, D15, D16, D18, D19, D20, D21, P4, Q10, Q11, Q12, Q14, Q15, Q9, R30, R31, R32, R33, R34, R35, R36, R37, R38, R39, R40, R41, R45, R46, R47, R48, R49, R50, R51, R52, R53, R54, R55, R56, R57, R58, R59, R60, R61, R62, R63, R64, TP1, TP2, TP3: moved to B.Cu
- J23: footprint MyModules:SJ1-3523N -> MyModules:CUI_SJ1-3523N
- U3, U4: footprint MyModules:R-78E-0.5 -> MyModules:CUI_VXO780XX-500
- moved R57 232.9 mm to (280.2, 91.5), turned to 180 degrees
- moved R60 229.6 mm to (275.5, 88.2), turned to 90 degrees
- moved R56 219.0 mm to (254.0, 67.8), turned to 270 degrees
- moved D18 217.2 mm to (251.8, 67.5), turned to 90 degrees
- moved D19 215.9 mm to (250.2, 67.5), turned to 270 degrees
- moved C18 215.8 mm to (260.5, 88.2), turned to 270 degrees
- moved R54 215.5 mm to (251.8, 71.0), turned to 90 degrees
- moved R55 213.9 mm to (251.8, 74.2), turned to 90 degrees
- moved R64 212.6 mm to (254.2, 82.2)
- moved R63 211.7 mm to (254.2, 84.2)
- moved D20 211.1 mm to (255.0, 87.2), turned to 90 degrees
- moved D21 209.8 mm to (253.5, 87.2), turned to 270 degrees
- moved R58 209.6 mm to (255.0, 91.0), turned to 90 degrees
- moved C17 209.1 mm to (255.8, 94.2)
- moved R62 208.3 mm to (250.5, 84.2)
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Other:
- board outline added: 280 x 38 mm

Commit message: first route complete
Parts:
- removed Q13: MMBT3904, MyModules:SOT23-132-JRL
- removed R42, R45: 10K, MyModules:SM0603-R-YAGEO
- removed R43, R44: 100K, MyModules:SM0603-R-YAGEO
- removed TP1: CONN_1, MyModules:TEST_POINT_LOOP_4592
- added R65: 0R, MyModules:SM0603-R-YAGEO, B.Cu at (98.6, 87.5)
- added R66: 0R, MyModules:SM0603-R-YAGEO, B.Cu at (143.4, 91.6)
- moved TP3 20.9 mm to (66.2, 92.0)
- moved C2 9.99 mm to (136.8, 93.8), turned to 180 degrees
- moved D1 4.27 mm to (87.0, 65.0), turned to 270 degrees
- moved R61 3.61 mm to (249.2, 92.2), turned to 90 degrees
- moved C3 3.58 mm to (101.5, 86.2), turned to 0 degrees
- moved C1 3.54 mm to (67.0, 79.0), turned to 0 degrees
- moved R48 3.34 mm to (224.5, 86.0), turned to 0 degrees
- moved D18 2.94 mm to (250.2, 70.0), turned to 270 degrees
- moved C9 2.62 mm to (31.9, 83.3), turned to 180 degrees
- moved R10 2.61 mm to (106.8, 62.5), turned to 0 degrees
- moved R11 2.61 mm to (106.8, 75.2), turned to 0 degrees
- moved R12 2.61 mm to (124.8, 62.5), turned to 0 degrees
- moved R13 2.61 mm to (124.8, 75.2), turned to 0 degrees
- moved R22 2.61 mm to (142.8, 62.2), turned to 0 degrees
- moved R23 2.61 mm to (142.8, 75.2), turned to 0 degrees
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Routing:
- net +5V: track 0.00 -> 328.6 mm, vias 0 -> 16
- net -V: track 0.00 -> 311.2 mm, vias 0 -> 4
- net +V: track 0.00 -> 272.0 mm, vias 0 -> 4
- net /OH: track 0.00 -> 68.9 mm
- net /CH: track 0.00 -> 64.4 mm
- net /CP: track 0.00 -> 63.4 mm
- net /MA: track 0.00 -> 59.2 mm
- net DIN_TEMPO_CLK: track 0.00 -> 58.3 mm
- net Net-(C16-Pad1): track 0.00 -> 55.0 mm
- net Net-(R1-Pad1): track 0.00 -> 51.0 mm
- net /CB: track 0.00 -> 50.2 mm
- net /HT: track 0.00 -> 48.7 mm
- net GND: track 0.00 -> 46.9 mm, vias 0 -> 10
- net /CY: track 0.00 -> 44.9 mm
- net Net-(C5-Pad1): track 0.00 -> 41.8 mm
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- added copper zone on B.Cu, net GND
- added copper zone on F.Cu, net GND
- added copper zone on B.Cu, net Net-(CON1-Pad1)
- added copper zone on F.Cu, net Net-(CON1-Pad1)
Other:
- outline, holes or cut-outs redrawn
- net class Default: clearance 0.2 -> 0.25; via_dia 0.6 -> 0.8
- net class POWER added: clearance 0.25, trace_width 0.35, via_dia 1, via_drill 0.5
- rule trace_clearance: 0.2 -> 0.25

Commit message: added insert on submix sum. put insert jack and headphone jack on daughter board
Parts:
- added J24: JACK_TRS_SWITCHED, MyModules:RA49B14B_SWITCHCRAFT, F.Cu at (307.0, 75.5)
- added P5: CONN_01X04, Pin_Headers:Pin_Header_Straight_1x04_Pitch2.54mm, B.Cu at (274.2, 65.5)
- added P6: CONN_01X04, Pin_Headers:Pin_Header_Straight_1x04_Pitch2.54mm, F.Cu at (311.0, 89.2)
- added P7: CONN_01X03, Pin_Headers:Pin_Header_Straight_1x03_Pitch2.54mm, B.Cu at (264.8, 88.5)
- added P8: CONN_01X03, Pin_Headers:Pin_Header_Straight_1x03_Pitch2.54mm, F.Cu at (324.2, 76.0)
- added R67: 120, Resistors_SMD:R_0805, B.Cu at (269.2, 62.0)
- J23: footprint MyModules:CUI_SJ1-3523N -> MyModules:CUI_SJ1-3513; moved to F.Cu
- moved J23 57.1 mm to (326.8, 59.2)
Connections:
- J21 pad 2: Net-(C16-Pad1) -> Net-(J21-Pad2)
- J23 pad 1: GND -> Net-(J23-Pad1)
- R54 pad 2: Net-(C16-Pad1) -> Net-(J21-Pad2)
- R56 pad 2: Net-(C16-Pad1) -> Net-(J21-Pad2)
- R63 pad 2: Net-(J23-Pad2) -> Net-(P7-Pad1)
- R64 pad 2: Net-(J23-Pad3) -> Net-(P7-Pad2)
Routing:
- net Net-(J24-Pad3): track 0.00 -> 40.8 mm
- net Net-(J24-Pad2): track 0.00 -> 33.8 mm
- net Net-(J21-Pad2): track 0.00 -> 33.2 mm
- net Net-(P7-Pad2): track 0.00 -> 21.4 mm, vias 0 -> 1
- net Net-(J23-Pad1): track 0.00 -> 17.8 mm
- net Net-(J23-Pad2): track 31.1 -> 14.7 mm, vias 1 -> 0
- net Net-(C16-Pad1): track 55.0 -> 68.6 mm
- net Net-(J24-Pad1): track 0.00 -> 13.0 mm
- net Net-(J24-Pad4): track 0.00 -> 12.4 mm
- net Net-(P7-Pad1): track 0.00 -> 12.0 mm, vias 0 -> 1
- net Net-(J23-Pad3): track 19.2 -> 10.5 mm, vias 1 -> 0
- net Net-(P5-Pad2): track 0.00 -> 4.51 mm
- net GND: track 46.9 -> 48.7 mm, vias 10 -> 11
- net Net-(J20-Pad3): track 16.4 -> 15.2 mm
Other:
- board size 280 x 38 mm -> 321.8 x 38 mm

Commit message: place silkscreen references
Parts:
- moved P8 13.2 mm to (324.2, 89.2)
Routing:
- net Net-(J23-Pad3): track 10.5 -> 24.0 mm
- net Net-(J23-Pad2): track 14.7 -> 27.9 mm
- net Net-(J23-Pad1): track 17.8 -> 31.1 mm
- net GND: track 48.7 -> 54.3 mm, vias 11 -> 14
- net +5V: track 328.6 -> 333.5 mm
- net -V: track 311.2 -> 313.8 mm
- net ISP_SCK: track 32.1 -> 32.9 mm
- net Net-(D20-Pad1): track 35.9 -> 36.6 mm

Commit message: more tweaking, almost ready to order
Parts:
- added HOLE-M3: VAL**, MyModules:HOLE-M3, F.Cu at (292.0, 84.8)
- added HOLE-M3: VAL**, MyModules:HOLE-M3, F.Cu at (292.0, 86.2)
- added HOLE-M3: VAL**, MyModules:HOLE-M3, F.Cu at (292.0, 87.8)
- added HOLE-M3: VAL**, MyModules:HOLE-M3, F.Cu at (292.0, 68.2)
- added HOLE-M3: VAL**, MyModules:HOLE-M3, F.Cu at (292.0, 66.8)
- added HOLE-M3: VAL**, MyModules:HOLE-M3, F.Cu at (292.0, 65.2)
- moved J23 5.00 mm to (321.8, 59.2)
- moved J24 5.00 mm to (302.0, 75.5)
- moved P6 5.00 mm to (306.0, 89.2)
- moved P8 5.00 mm to (319.2, 89.2)
- moved R57 4.72 mm to (275.6, 92.3), turned to 270 degrees
Routing:
- net Net-(R57-Pad2): track 23.7 -> 19.3 mm
- net Net-(P4-Pad2): track 3.06 -> 7.48 mm
- net Net-(J24-Pad3): track 40.8 -> 44.4 mm
- net Net-(J24-Pad4): track 12.4 -> 13.6 mm
- net Net-(J24-Pad2): track 33.8 -> 32.7 mm
- net ISP_MOSI: track 33.3 -> 34.2 mm
- net Net-(J24-Pad1): track 13.0 -> 13.8 mm
Other:
- board size 321.8 x 38 mm -> 316.8 x 38 mm
- board text added: "A1"
- board text added: "A2"
- board text added: "A3"
- board text added: "A4"
- board text added: "B1"
- board text added: "B2"
- board text added: "B3"
- board text added: "C1"
- board text added: "C2"
- board text added: "C3"
- board text added: "DIN EXPANDER"
- board text added: "ISP"
- board text added: "POWER"
- board text added: "R"
- board text added: "S"
- board text added: "T"
- board text added: "−12V"

Commit message: first prototype PCB ordered
Parts:
- removed R65, R66: 0R, MyModules:SM0603-R-YAGEO
- added G***: LOGO, LOGO, B.Cu at (28.2, 63.2)
- added G***: LOGO, LOGO, F.Cu at (28.2, 63.2)
- added G***: LOGO, LOGO, B.Cu at (315.3, 77.3)
- added P9: CONN_01X03, Pin_Headers:Pin_Header_Straight_1x03_Pitch2.54mm, B.Cu at (144.5, 86.5)
- added Q13: MMBT3904, MyModules:SOT23-132-JRL, B.Cu at (153.5, 86.5)
- added R42: 10K, MyModules:SM0603-R-YAGEO, B.Cu at (159.2, 83.8)
- added R43: 100K, MyModules:SM0603-R-YAGEO, B.Cu at (159.2, 85.5)
- added R44: 100K, MyModules:SM0603-R-YAGEO, B.Cu at (156.8, 86.5)
- added R45: 10K, MyModules:SM0603-R-YAGEO, B.Cu at (156.0, 83.8)
Connections:
- U2 pad 3: Net-(U2-Pad3) -> GND
- U2 pad 4: Net-(U2-Pad4) -> GND
- U2 pad 5: Net-(U2-Pad5) -> GND
Routing:
- net ~RESET: track 0.00 -> 56.2 mm, vias 0 -> 2
- net /~CE: track 7.57 -> 62.2 mm, vias 0 -> 2
- net GND: track 54.3 -> 88.0 mm, vias 14 -> 19
- net Net-(P9-Pad3): track 0.00 -> 7.31 mm
- net Net-(CON1-Pad1): track 7.05 -> 0.00 mm
- net /CB: track 50.2 -> 54.9 mm
- net Net-(Q13-Pad1): track 0.00 -> 3.73 mm
- net /CP: track 63.4 -> 64.8 mm
- net /CH: track 64.4 -> 63.4 mm
- net /RS: track 40.8 -> 39.9 mm
- net /MA: track 59.2 -> 58.4 mm
- net +5V: track 333.5 -> 333.6 mm, vias 16 -> 17
Other:
- rule pad_to_mask_clearance: 0.2 -> 0.05
- board text added: "880 case board r1.0 2/2019"
- board text added: "GND"
- board text added: "RESET"
- board text added: "~CE"
