File: _autosave-880_enclosure_subboards.kicad_pcb (KiCad board)
At the start: 2 copper layers, 54.3 x 38 mm, 16 parts, among them J23 JACK_STEREO, J24 JACK_TRS_SWITCHED, J25 JACK_STEREO, P10 CONN_01X02, P11 CONN_01X03, P6 CONN_01X04, P8 CONN_01X03, SW1 SPST

Commit message: v1.1 ordered plus sub boards
Other:
- board text added: "880ENC 6/2019"
Changed lines of the file:
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@@
     (links 13)
     (no_connects 0)
-    (area 296.949999 57.449999 351.304027 95.550933)
+    (area 296.949999 50.740199 351.304027 95.550933)
     (thickness 1.6)
-    (drawings 41)
+    (drawings 42)
     (tracks 51)
     (zones 0)
@@
     )
   )
+  (gr_text "880ENC 6/2019" (at 303.5 94.25) (layer B.SilkS)
+    (effects (font (size 1 1) (thickness 0.15)) (justify mirror))
+  )
   (gr_line (start 334.25 86.75) (end 334.25 77.75) (layer Edge.Cuts) (width 0.1))
