File: 880_case.sch (KiCad schematic (older format))
At the start: 173 parts, among them CON1 BARREL_JACK, J1 RUN/STOP, J10 RS IN, J11 CP IN, J12 MA IN, J13 CB IN, J14 CY IN, J15 OH IN, J16 CH IN, J17 IN 1, J18 IN 2, J19 IN 3, J2 SYNC24 CLK, J20 IN 4, J21 MULT IN, J22 SUM, J23 JACK_STEREO, J24 JACK_TRS_SWITCHED, J25 JACK_STEREO, J3 ASSIGN 1, J4 ASSIGN 2, J5 BD IN, J6 SD IN, J7 LT IN, J8 MT IN, J9 HT IN, P1 CONN_02X03, P10 CONN_01X02, P11 CONN_01X03, P2 CONN_01X02, P3 CONN_02X08, P4 CONN_01X03, P5 CONN_01X04, P6 CONN_01X04, P7 CONN_01X03, P8 CONN_01X03, Q1 MMBT3904, Q10 MMBT3904, Q11 MMBT3904, Q12 MMBT3904, Q14 C945, Q15 A733, Q2 MMBT3904, Q3 MMBT3904, Q4 MMBT3904, Q5 MMBT3904, Q6 MMBT3904, Q7 MMBT3904, Q8 MMBT3904, Q9 MMBT3904, SW1 SPST, U1 74HC165, U2 74HC165, U3 VX078-500, U4 VX078-500, U5 4558, U6 4558, U7 74HCT1G125GV, X1 MIDI OUT, X2 SYNC24

Commit message: getting ready to panelize for production
Changed lines of the file:
@@
 Comment4 ""
 $EndDescr
-Text GLabel 12150 7375 2    50   Input ~ 0
+Text GLabel 12625 8150 2    50   Input ~ 0
 ISP_MOSI
-Text GLabel 11650 7275 0    50   Output ~ 0
+Text GLabel 11175 7275 0    50   Output ~ 0
 ISP_MISO
-Text GLabel 11650 7375 0    50   BiDi ~ 0
+Text GLabel 11200 7375 0    50   BiDi ~ 0
 ISP_SCK
 $Comp
@@
 Text GLabel 4400 4650 0    50   BiDi ~ 0
 DIN_FILL
-Text GLabel 1900 4125 0    50   BiDi ~ 0
+Text GLabel 1900 4125 0    60   BiDi ~ 0
 DIN_TEMPO_CLK
 Wire Wire Line
@@
 	1    0    0    -1
 $EndComp
+Wire Wire Line
+	11200 7375 11650 7375
+Wire Wire Line
+	11175 7275 11650 7275
+Wire Wire Line
+	12550 7375 12550 8150
+Wire Wire Line
+	12550 8150 12625 8150
+Wire Wire Line
+	12150 7375 12550 7375
 $EndSCHEMATC
