File: 880_enclosure_panelized.kicad_pcb (KiCad board)
At the start: 4 copper layers, 279.5 x 38 mm, 164 parts, among them CON1 BARREL_JACK, J1 RUN/STOP, J10 RS IN, J11 CP IN, J12 MA IN, J13 CB IN, J14 CY IN, J15 OH IN, J16 CH IN, J17 IN 1, J18 IN 2, J19 IN 3, J2 SYNC24 CLK, J20 IN 4, J21 MULT IN, J22 SUM, J3 ASSIGN 1, J4 ASSIGN 2, J5 BD IN, J6 SD IN, J7 LT IN, J8 MT IN, J9 HT IN, P1 CONN_02X03, P2 CONN_01X02, P3 CONN_02X08, P4 CONN_01X03, P5 CONN_01X04, P7 CONN_01X03, Q1 MMBT3904, Q10 MMBT3904, Q11 MMBT3904, Q12 MMBT3904, Q14 C945, Q15 A733, Q2 MMBT3904, Q3 MMBT3904, Q4 MMBT3904, Q5 MMBT3904, Q6 MMBT3904, Q7 MMBT3904, Q8 MMBT3904, Q9 MMBT3904, U1 74HC165, U2 74HC165, U3 VX078-500, U4 VX078-500, U5 4558, U6 4558, U7 74HC1G125, X1 MIDI OUT, X2 SYNC24

Commit message: getting ready to panelize for production
Parts:
- added REF**: fiducial-1mm, MyModules:fiducial-1mm, B.Cu at (289.0, 93.0)
- added REF**: fiducial-1mm, MyModules:fiducial-1mm, B.Cu at (14.5, 60.0)
- P1: footprint w_conn_strip:vasch_strip_3x2 -> w_conn_strip:vasch_strip_4x2
- moved R1 6.50 mm to (78.8, 84.2), turned to 0 degrees
- moved P1 1.27 mm to (86.7, 90.2)
Routing:
- net GNDD: track 79.9 -> 113.6 mm, vias 7 -> 8
- net UART_TX: track 7.42 -> 12.8 mm
- net Net-(R1-Pad1): track 51.0 -> 46.2 mm
- net GND: track 51.2 -> 54.7 mm
Other:
- board text added: "880ENC MAIN BOARD r1.3 2/2020"
- board text removed: "880ENC MAIN BOARD r1.2 9/2019"

Commit message: first update in a long while. this version and gone through production
Parts:
- added C1: 0.01µ, MyModules:SM0603-C-MURATA, B.Cu at (67.0, 193.0)
- added C1: 0.01µ, MyModules:SM0603-C-MURATA, B.Cu at (67.0, 155.0)
- added C1: 0.01µ, MyModules:SM0603-C-MURATA, B.Cu at (67.0, 117.0)
- added C10: 22µF, Capacitors_SMD:C_1206, B.Cu at (42.0, 159.3)
- added C10: 22µF, Capacitors_SMD:C_1206, B.Cu at (42.0, 197.3)
- added C10: 22µF, Capacitors_SMD:C_1206, B.Cu at (42.0, 121.3)
- added C11: 1μ, Capacitors_SMD:CP_Elec_4x5.3, B.Cu at (226.2, 205.0)
- added C11: 1μ, Capacitors_SMD:CP_Elec_4x5.3, B.Cu at (226.2, 167.0)
- added C11: 1μ, Capacitors_SMD:CP_Elec_4x5.3, B.Cu at (226.2, 129.0)
- added C12: 220p, MyModules:SM0603-C-MURATA, B.Cu at (231.5, 207.5)
- added C12: 220p, MyModules:SM0603-C-MURATA, B.Cu at (231.5, 169.5)
- added C12: 220p, MyModules:SM0603-C-MURATA, B.Cu at (231.5, 131.5)
- added C13: 0.1µ, MyModules:SM0603-C-MURATA, B.Cu at (236.8, 206.3)
- added C13: 0.1µ, MyModules:SM0603-C-MURATA, B.Cu at (236.8, 168.3)
- added C13: 0.1µ, MyModules:SM0603-C-MURATA, B.Cu at (236.8, 130.3)
- added C14: 0.1µ, MyModules:SM0603-C-MURATA, B.Cu at (231.2, 200.8)
- added C14: 0.1µ, MyModules:SM0603-C-MURATA, B.Cu at (231.2, 162.8)
- added C14: 0.1µ, MyModules:SM0603-C-MURATA, B.Cu at (231.2, 124.8)
- added C15: 1µ, Capacitors_SMD:C_0805, B.Cu at (122.2, 189.8)
- added C15: 1µ, Capacitors_SMD:C_0805, B.Cu at (122.2, 151.8)
- added C15: 1µ, Capacitors_SMD:C_0805, B.Cu at (122.2, 113.8)
- added C16: 220p, MyModules:SM0603-C-MURATA, B.Cu at (234.8, 161.2)
- added C16: 220p, MyModules:SM0603-C-MURATA, B.Cu at (234.8, 199.2)
- added C16: 220p, MyModules:SM0603-C-MURATA, B.Cu at (234.8, 123.2)
- added C17: 0.1µ, MyModules:SM0603-C-MURATA, B.Cu at (269.2, 173.4)
- added C17: 0.1µ, MyModules:SM0603-C-MURATA, B.Cu at (269.2, 135.4)
- added C17: 0.1µ, MyModules:SM0603-C-MURATA, B.Cu at (269.2, 97.4)
- added C18: 0.1µ, MyModules:SM0603-C-MURATA, B.Cu at (264.8, 178.9)
- added C18: 0.1µ, MyModules:SM0603-C-MURATA, B.Cu at (264.8, 140.9)
- added C18: 0.1µ, MyModules:SM0603-C-MURATA, B.Cu at (264.8, 103.0)
- added C19: 0.1µ, MyModules:SM0603-C-MURATA, B.Cu at (120.5, 189.8)
- added C19: 0.1µ, MyModules:SM0603-C-MURATA, B.Cu at (120.5, 151.8)
- added C19: 0.1µ, MyModules:SM0603-C-MURATA, B.Cu at (120.5, 113.8)
- added C2: 0.1µ, MyModules:SM0603-C-MURATA, B.Cu at (136.8, 207.8)
- added C2: 0.1µ, MyModules:SM0603-C-MURATA, B.Cu at (136.8, 169.8)
- added C2: 0.1µ, MyModules:SM0603-C-MURATA, B.Cu at (136.8, 131.8)
- added C20: 0.1µ, MyModules:SM0603-C-MURATA, B.Cu at (140.9, 200.5)
- added C20: 0.1µ, MyModules:SM0603-C-MURATA, B.Cu at (140.9, 162.5)
- added C20: 0.1µ, MyModules:SM0603-C-MURATA, B.Cu at (140.9, 124.5)
- added C23: 1μ, Capacitors_SMD:CP_Elec_4x5.3, B.Cu at (240.5, 161.8)
- added C23: 1μ, Capacitors_SMD:CP_Elec_4x5.3, B.Cu at (240.5, 199.8)
- added C23: 1μ, Capacitors_SMD:CP_Elec_4x5.3, B.Cu at (240.5, 123.8)
- added C3: 0.1µ, MyModules:SM0603-C-MURATA, B.Cu at (101.5, 200.2)
- added C3: 0.1µ, MyModules:SM0603-C-MURATA, B.Cu at (101.5, 162.2)
- added C3: 0.1µ, MyModules:SM0603-C-MURATA, B.Cu at (101.5, 124.2)
- added C4: 4.7µ, Capacitors_SMD:C_1206, B.Cu at (27.0, 191.5)
- added C4: 4.7µ, Capacitors_SMD:C_1206, B.Cu at (27.0, 153.5)
- added C4: 4.7µ, Capacitors_SMD:C_1206, B.Cu at (27.0, 115.5)
- added C5: 10µ, Capacitors_SMD:C_1206, B.Cu at (23.0, 199.0)
- added C5: 10µ, Capacitors_SMD:C_1206, B.Cu at (23.0, 161.0)
- added C5: 10µ, Capacitors_SMD:C_1206, B.Cu at (23.0, 123.0)
- added C6: 10µ, Capacitors_SMD:C_1206, B.Cu at (71.0, 199.0)
- added C6: 10µ, Capacitors_SMD:C_1206, B.Cu at (71.0, 161.0)
- added C6: 10µ, Capacitors_SMD:C_1206, B.Cu at (71.0, 123.0)
- added C7: 22µF, Capacitors_SMD:C_1206, B.Cu at (23.0, 204.0)
- added C7: 22µF, Capacitors_SMD:C_1206, B.Cu at (23.0, 166.0)
- added C7: 22µF, Capacitors_SMD:C_1206, B.Cu at (23.0, 128.0)
- added C8: 22µF, Capacitors_SMD:C_1206, B.Cu at (71.0, 204.5)
- added C8: 22µF, Capacitors_SMD:C_1206, B.Cu at (71.0, 166.5)
- added C8: 22µF, Capacitors_SMD:C_1206, B.Cu at (71.0, 128.5)
- added C9: 22µF, Capacitors_SMD:C_1206, B.Cu at (31.9, 159.3)
- added C9: 22µF, Capacitors_SMD:C_1206, B.Cu at (31.9, 197.3)
- added C9: 22µF, Capacitors_SMD:C_1206, B.Cu at (31.9, 121.3)
- added CON1: BARREL_JACK, MyModules:712A-DC-JACK, F.Cu at (20.2, 186.2)
- added CON1: BARREL_JACK, MyModules:712A-DC-JACK, F.Cu at (20.2, 148.2)
- added CON1: BARREL_JACK, MyModules:712A-DC-JACK, F.Cu at (20.2, 110.2)
- added D1: NSR0530HT1G, MyModules:SOD323-C1A2, B.Cu at (87.0, 179.0)
- added D1: NSR0530HT1G, MyModules:SOD323-C1A2, B.Cu at (87.0, 141.0)
- added D1: NSR0530HT1G, MyModules:SOD323-C1A2, B.Cu at (87.0, 103.0)
- added D10: 1N4148, MyModules:SOD323-C1A2, B.Cu at (143.0, 187.8)
- added D10: 1N4148, MyModules:SOD323-C1A2, B.Cu at (143.0, 149.8)
- added D10: 1N4148, MyModules:SOD323-C1A2, B.Cu at (143.0, 111.8)
- added D11: 1N4148, MyModules:SOD323-C1A2, B.Cu at (161.0, 174.8)
- added D11: 1N4148, MyModules:SOD323-C1A2, B.Cu at (161.0, 136.8)
- added D11: 1N4148, MyModules:SOD323-C1A2, B.Cu at (161.0, 98.8)
- added D12: 1N4148, MyModules:SOD323-C1A2, B.Cu at (161.0, 187.8)
- added D12: 1N4148, MyModules:SOD323-C1A2, B.Cu at (161.0, 149.8)
- added D12: 1N4148, MyModules:SOD323-C1A2, B.Cu at (161.0, 111.8)
- added D13: 1N4148, MyModules:SOD323-C1A2, B.Cu at (179.0, 174.8)
- added D13: 1N4148, MyModules:SOD323-C1A2, B.Cu at (179.0, 136.8)
- added D13: 1N4148, MyModules:SOD323-C1A2, B.Cu at (179.0, 98.8)
- added D14: 1N4148, MyModules:SOD323-C1A2, B.Cu at (179.0, 187.8)
- added D14: 1N4148, MyModules:SOD323-C1A2, B.Cu at (179.0, 149.8)
- added D14: 1N4148, MyModules:SOD323-C1A2, B.Cu at (179.0, 111.8)
- added D15: 1N4148, MyModules:SOD323-C1A2, B.Cu at (197.0, 174.8)
- added D15: 1N4148, MyModules:SOD323-C1A2, B.Cu at (197.0, 136.8)
- added D15: 1N4148, MyModules:SOD323-C1A2, B.Cu at (197.0, 98.8)
- added D16: 1N4148, MyModules:SOD323-C1A2, B.Cu at (197.0, 187.8)
- added D16: 1N4148, MyModules:SOD323-C1A2, B.Cu at (197.0, 149.8)
- added D16: 1N4148, MyModules:SOD323-C1A2, B.Cu at (197.0, 111.8)
- added D17: MBRS240LT3G, MyModules:SMB-1C2A, B.Cu at (20.5, 194.0)
- added D17: MBRS240LT3G, MyModules:SMB-1C2A, B.Cu at (20.5, 156.0)
- added D17: MBRS240LT3G, MyModules:SMB-1C2A, B.Cu at (20.5, 118.0)
- added D18: 1N4148, MyModules:SOD323-C1A2, B.Cu at (250.2, 184.0)
- added D18: 1N4148, MyModules:SOD323-C1A2, B.Cu at (250.2, 146.0)
- added D18: 1N4148, MyModules:SOD323-C1A2, B.Cu at (250.2, 108.0)
- added D19: 1N4148, MyModules:SOD323-C1A2, B.Cu at (251.8, 181.5)
- added D19: 1N4148, MyModules:SOD323-C1A2, B.Cu at (251.8, 143.5)
- added D19: 1N4148, MyModules:SOD323-C1A2, B.Cu at (251.8, 105.5)
- added D2: NSR0530HT1G, MyModules:SOD323-C1A2, B.Cu at (87.0, 137.0)
- added D2: NSR0530HT1G, MyModules:SOD323-C1A2, B.Cu at (87.0, 175.0)
- added D2: NSR0530HT1G, MyModules:SOD323-C1A2, B.Cu at (87.0, 99.0)
- added D20: 1N4148, MyModules:SOD323-C1A2, B.Cu at (270.2, 141.9)
- added D20: 1N4148, MyModules:SOD323-C1A2, B.Cu at (270.2, 179.9)
- added D20: 1N4148, MyModules:SOD323-C1A2, B.Cu at (270.2, 104.0)
- added D21: 1N4148, MyModules:SOD323-C1A2, B.Cu at (271.8, 141.9)
- added D21: 1N4148, MyModules:SOD323-C1A2, B.Cu at (271.8, 179.9)
- added D21: 1N4148, MyModules:SOD323-C1A2, B.Cu at (271.8, 104.0)
- added D3: NSR0530HT1G, MyModules:SOD323-C1A2, B.Cu at (88.5, 188.2)
- added D3: NSR0530HT1G, MyModules:SOD323-C1A2, B.Cu at (88.5, 150.2)
- added D3: NSR0530HT1G, MyModules:SOD323-C1A2, B.Cu at (88.5, 112.2)
- added D4: NSR0530HT1G, MyModules:SOD323-C1A2, B.Cu at (87.0, 188.2)
- added D4: NSR0530HT1G, MyModules:SOD323-C1A2, B.Cu at (87.0, 150.2)
- added D4: NSR0530HT1G, MyModules:SOD323-C1A2, B.Cu at (87.0, 112.2)
- added D5: 1N4148, MyModules:SOD323-C1A2, B.Cu at (107.0, 175.0)
- added D5: 1N4148, MyModules:SOD323-C1A2, B.Cu at (107.0, 137.0)
- added D5: 1N4148, MyModules:SOD323-C1A2, B.Cu at (107.0, 99.0)
- added D6: 1N4148, MyModules:SOD323-C1A2, B.Cu at (107.0, 187.8)
- added D6: 1N4148, MyModules:SOD323-C1A2, B.Cu at (107.0, 149.8)
- added D6: 1N4148, MyModules:SOD323-C1A2, B.Cu at (107.0, 111.8)
- added D7: 1N4148, MyModules:SOD323-C1A2, B.Cu at (125.0, 175.0)
- added D7: 1N4148, MyModules:SOD323-C1A2, B.Cu at (125.0, 137.0)
- added D7: 1N4148, MyModules:SOD323-C1A2, B.Cu at (125.0, 99.0)
- added D8: 1N4148, MyModules:SOD323-C1A2, B.Cu at (125.0, 187.8)
- added D8: 1N4148, MyModules:SOD323-C1A2, B.Cu at (125.0, 149.8)
- added D8: 1N4148, MyModules:SOD323-C1A2, B.Cu at (125.0, 111.8)
- added D9: 1N4148, MyModules:SOD323-C1A2, B.Cu at (143.0, 174.8)
- added D9: 1N4148, MyModules:SOD323-C1A2, B.Cu at (143.0, 136.8)
- added D9: 1N4148, MyModules:SOD323-C1A2, B.Cu at (143.0, 98.8)
- added G***: LOGO, w_logo:Logo_silk_polarity_center_10x2.8mm, F.Cu at (20.0, 178.0)
- added G***: LOGO, LOGO, F.Cu at (151.0, 206.0)
- added G***: LOGO, LOGO, F.Cu at (151.0, 168.0)
- added G***: LOGO, LOGO, F.Cu at (151.0, 130.0)
- added G***: LOGO, LOGO, F.Cu at (151.0, 92.0)
- added G***: LOGO, w_logo:Logo_silk_Lead-Free_5x5mm, F.Cu at (202.0, 89.5)
- added G***: LOGO, w_logo:Logo_silk_polarity_center_10x2.8mm, F.Cu at (20.0, 64.0)
- added G***: LOGO, w_logo:Logo_silk_ROHS_10x5.6mm, F.Cu at (194.0, 89.0)
- added G***: LOGO, w_logo:Logo_silk_polarity_center_10x2.8mm, F.Cu at (20.0, 140.0)
- added G***: LOGO, w_logo:Logo_silk_polarity_center_10x2.8mm, F.Cu at (20.0, 102.0)
- added G***: LOGO, w_logo:Logo_silk_ROHS_10x5.6mm, F.Cu at (194.0, 203.0)
- added G***: LOGO, w_logo:Logo_silk_Lead-Free_5x5mm, F.Cu at (202.0, 203.5)
- added G***: LOGO, w_logo:Logo_silk_ROHS_10x5.6mm, F.Cu at (194.0, 165.0)
- added G***: LOGO, w_logo:Logo_silk_Lead-Free_5x5mm, F.Cu at (202.0, 165.5)
- added G***: LOGO, w_logo:Logo_silk_ROHS_10x5.6mm, F.Cu at (194.0, 127.0)
- added G***: LOGO, w_logo:Logo_silk_Lead-Free_5x5mm, F.Cu at (202.0, 127.5)
- added HOLE-M3: VAL**, MyModules:HOLE-M3, F.Cu at (15.0, 212.5)
- added HOLE-M3: VAL**, MyModules:HOLE-M3, F.Cu at (288.5, 212.5)
- added HOLE-M3: VAL**, MyModules:HOLE-M3, F.Cu at (288.5, 54.5)
- added HOLE-M3: VAL**, MyModules:HOLE-M3, F.Cu at (15.0, 54.5)
- added ISP1: CONN_02X03, w_conn_strip:vasch_strip_3x2, B.Cu at (119.8, 204.2)
- added ISP1: CONN_02X03, w_conn_strip:vasch_strip_3x2, B.Cu at (119.8, 166.2)
- added ISP1: CONN_02X03, w_conn_strip:vasch_strip_3x2, B.Cu at (119.8, 128.2)
- added J1: RUN/STOP, MyModules:PJ-301B-JACK-SLOTS, F.Cu at (79.0, 191.0)
- added J1: RUN/STOP, MyModules:PJ-301B-JACK-SLOTS, F.Cu at (79.0, 153.0)
- added J1: RUN/STOP, MyModules:PJ-301B-JACK-SLOTS, F.Cu at (79.0, 115.0)
- added J10: RS IN, MyModules:PJ-301B-JACK-SLOTS, F.Cu at (151.0, 191.0)
- added J10: RS IN, MyModules:PJ-301B-JACK-SLOTS, F.Cu at (151.0, 153.0)
- added J10: RS IN, MyModules:PJ-301B-JACK-SLOTS, F.Cu at (151.0, 115.0)
- added J11: CP IN, MyModules:PJ-301B-JACK-SLOTS, F.Cu at (169.0, 140.0)
- added J11: CP IN, MyModules:PJ-301B-JACK-SLOTS, F.Cu at (169.0, 178.0)
- added J11: CP IN, MyModules:PJ-301B-JACK-SLOTS, F.Cu at (169.0, 102.0)
- added J12: MA IN, MyModules:PJ-301B-JACK-SLOTS, F.Cu at (169.0, 153.0)
- added J12: MA IN, MyModules:PJ-301B-JACK-SLOTS, F.Cu at (169.0, 191.0)
- added J12: MA IN, MyModules:PJ-301B-JACK-SLOTS, F.Cu at (169.0, 115.0)
- added J13: CB IN, MyModules:PJ-301B-JACK-SLOTS, F.Cu at (187.0, 140.0)
- added J13: CB IN, MyModules:PJ-301B-JACK-SLOTS, F.Cu at (187.0, 178.0)
- added J13: CB IN, MyModules:PJ-301B-JACK-SLOTS, F.Cu at (187.0, 102.0)
- added J14: CY IN, MyModules:PJ-301B-JACK-SLOTS, F.Cu at (187.0, 153.0)
- added J14: CY IN, MyModules:PJ-301B-JACK-SLOTS, F.Cu at (187.0, 191.0)
- added J14: CY IN, MyModules:PJ-301B-JACK-SLOTS, F.Cu at (187.0, 115.0)
- added J15: OH IN, MyModules:PJ-301B-JACK-SLOTS, F.Cu at (205.0, 140.0)
- added J15: OH IN, MyModules:PJ-301B-JACK-SLOTS, F.Cu at (205.0, 178.0)
- added J15: OH IN, MyModules:PJ-301B-JACK-SLOTS, F.Cu at (205.0, 102.0)
- added J16: CH IN, MyModules:PJ-301B-JACK-SLOTS, F.Cu at (205.0, 191.0)
- added J16: CH IN, MyModules:PJ-301B-JACK-SLOTS, F.Cu at (205.0, 153.0)
- added J16: CH IN, MyModules:PJ-301B-JACK-SLOTS, F.Cu at (205.0, 115.0)
- added J17: IN 1, MyModules:PJ-301B-JACK-SLOTS, F.Cu at (223.0, 140.0)
- added J17: IN 1, MyModules:PJ-301B-JACK-SLOTS, F.Cu at (223.0, 178.0)
- added J17: IN 1, MyModules:PJ-301B-JACK-SLOTS, F.Cu at (223.0, 102.0)
- added J18: IN 2, MyModules:PJ-301B-JACK-SLOTS, F.Cu at (223.0, 153.0)
- added J18: IN 2, MyModules:PJ-301B-JACK-SLOTS, F.Cu at (223.0, 191.0)
- added J18: IN 2, MyModules:PJ-301B-JACK-SLOTS, F.Cu at (223.0, 115.0)
- added J19: IN 3, MyModules:PJ-301B-JACK-SLOTS, F.Cu at (241.0, 140.0)
- added J19: IN 3, MyModules:PJ-301B-JACK-SLOTS, F.Cu at (241.0, 178.0)
- added J19: IN 3, MyModules:PJ-301B-JACK-SLOTS, F.Cu at (241.0, 102.0)
- added J2: SYNC24 CLK, MyModules:PJ-301B-JACK-SLOTS, F.Cu at (79.0, 178.0)
- added J2: SYNC24 CLK, MyModules:PJ-301B-JACK-SLOTS, F.Cu at (79.0, 140.0)
- added J2: SYNC24 CLK, MyModules:PJ-301B-JACK-SLOTS, F.Cu at (79.0, 102.0)
- added J20: IN 4, MyModules:PJ-301B-JACK-SLOTS, F.Cu at (241.0, 191.0)
- added J20: IN 4, MyModules:PJ-301B-JACK-SLOTS, F.Cu at (241.0, 153.0)
- added J20: IN 4, MyModules:PJ-301B-JACK-SLOTS, F.Cu at (241.0, 115.0)
- added J21: MULT IN, MyModules:PJ-301B-JACK-SLOTS, F.Cu at (259.0, 153.0)
- added J21: MULT IN, MyModules:PJ-301B-JACK-SLOTS, F.Cu at (259.0, 191.0)
- added J21: MULT IN, MyModules:PJ-301B-JACK-SLOTS, F.Cu at (259.0, 115.0)
- added J22: SUM, MyModules:PJ-301B-JACK-SLOTS, F.Cu at (259.0, 140.0)
- added J22: SUM, MyModules:PJ-301B-JACK-SLOTS, F.Cu at (259.0, 178.0)
- added J22: SUM, MyModules:PJ-301B-JACK-SLOTS, F.Cu at (259.0, 102.0)
- added J3: ASSIGN 1, MyModules:PJ-301B-JACK-SLOTS, F.Cu at (97.0, 140.0)
- added J3: ASSIGN 1, MyModules:PJ-301B-JACK-SLOTS, F.Cu at (97.0, 178.0)
- added J3: ASSIGN 1, MyModules:PJ-301B-JACK-SLOTS, F.Cu at (97.0, 102.0)
- added J4: ASSIGN 2, MyModules:PJ-301B-JACK-SLOTS, F.Cu at (97.0, 153.0)
- added J4: ASSIGN 2, MyModules:PJ-301B-JACK-SLOTS, F.Cu at (97.0, 191.0)
- added J4: ASSIGN 2, MyModules:PJ-301B-JACK-SLOTS, F.Cu at (97.0, 115.0)
- added J5: BD IN, MyModules:PJ-301B-JACK-SLOTS, F.Cu at (115.0, 140.0)
- added J5: BD IN, MyModules:PJ-301B-JACK-SLOTS, F.Cu at (115.0, 178.0)
- added J5: BD IN, MyModules:PJ-301B-JACK-SLOTS, F.Cu at (115.0, 102.0)
- added J6: SD IN, MyModules:PJ-301B-JACK-SLOTS, F.Cu at (115.0, 153.0)
- added J6: SD IN, MyModules:PJ-301B-JACK-SLOTS, F.Cu at (115.0, 191.0)
- added J6: SD IN, MyModules:PJ-301B-JACK-SLOTS, F.Cu at (115.0, 115.0)
- added J7: LT IN, MyModules:PJ-301B-JACK-SLOTS, F.Cu at (133.0, 140.0)
- added J7: LT IN, MyModules:PJ-301B-JACK-SLOTS, F.Cu at (133.0, 178.0)
- added J7: LT IN, MyModules:PJ-301B-JACK-SLOTS, F.Cu at (133.0, 102.0)
- added J8: MT IN, MyModules:PJ-301B-JACK-SLOTS, F.Cu at (133.0, 153.0)
- added J8: MT IN, MyModules:PJ-301B-JACK-SLOTS, F.Cu at (133.0, 191.0)
- added J8: MT IN, MyModules:PJ-301B-JACK-SLOTS, F.Cu at (133.0, 115.0)
- added J9: HT IN, MyModules:PJ-301B-JACK-SLOTS, F.Cu at (151.0, 140.0)
- added J9: HT IN, MyModules:PJ-301B-JACK-SLOTS, F.Cu at (151.0, 178.0)
- added J9: HT IN, MyModules:PJ-301B-JACK-SLOTS, F.Cu at (151.0, 102.0)
- added L1: 12µH, MyModules:SM0805-HAND, B.Cu at (25.5, 195.0)
- added L1: 12µH, MyModules:SM0805-HAND, B.Cu at (25.5, 157.0)
- added L1: 12µH, MyModules:SM0805-HAND, B.Cu at (25.5, 119.0)
- added L2: 10µH, MyModules:SM0805-HAND, B.Cu at (59.2, 199.2)
- added L2: 10µH, MyModules:SM0805-HAND, B.Cu at (59.2, 161.2)
- added L2: 10µH, MyModules:SM0805-HAND, B.Cu at (59.2, 123.2)
- added L3: 10µH, MyModules:SM0805-HAND, B.Cu at (25.5, 204.4)
- added L3: 10µH, MyModules:SM0805-HAND, B.Cu at (25.5, 166.4)
- added L3: 10µH, MyModules:SM0805-HAND, B.Cu at (25.5, 128.4)
- added L4: 10µH, MyModules:SM0805-HAND, B.Cu at (59.2, 204.1)
- added L4: 10µH, MyModules:SM0805-HAND, B.Cu at (59.2, 166.1)
- added L4: 10µH, MyModules:SM0805-HAND, B.Cu at (59.2, 128.1)
- added P1: CONN_02X03, w_conn_strip:vasch_strip_4x2, B.Cu at (86.7, 204.2)
- added P1: CONN_02X03, w_conn_strip:vasch_strip_4x2, B.Cu at (86.7, 166.2)
- added P1: CONN_02X03, w_conn_strip:vasch_strip_4x2, B.Cu at (86.7, 128.2)
- added P2: CONN_01X02, Pin_Headers:Pin_Header_Straight_1x02_Pitch2.54mm, B.Cu at (14.5, 191.5)
- added P2: CONN_01X02, Pin_Headers:Pin_Header_Straight_1x02_Pitch2.54mm, B.Cu at (14.5, 153.5)
- added P2: CONN_01X02, Pin_Headers:Pin_Header_Straight_1x02_Pitch2.54mm, B.Cu at (14.5, 115.5)
- added P3: CONN_02X08, w_conn_strip:vasch_strip_8x2, B.Cu at (42.5, 204.2)
- added P3: CONN_02X08, w_conn_strip:vasch_strip_8x2, B.Cu at (42.5, 166.2)
- added P3: CONN_02X08, w_conn_strip:vasch_strip_8x2, B.Cu at (42.5, 128.2)
- added P4: CONN_01X03, Pin_Headers:Pin_Header_Straight_1x03_Pitch2.54mm, B.Cu at (284.5, 202.9)
- added P4: CONN_01X03, Pin_Headers:Pin_Header_Straight_1x03_Pitch2.54mm, B.Cu at (284.5, 164.9)
- added P4: CONN_01X03, Pin_Headers:Pin_Header_Straight_1x03_Pitch2.54mm, B.Cu at (284.5, 126.9)
- added P5: CONN_01X04, Pin_Headers:Pin_Header_Straight_1x04_Pitch2.54mm, B.Cu at (264.2, 202.9)
- added P5: CONN_01X04, Pin_Headers:Pin_Header_Straight_1x04_Pitch2.54mm, B.Cu at (264.2, 164.9)
- added P5: CONN_01X04, Pin_Headers:Pin_Header_Straight_1x04_Pitch2.54mm, B.Cu at (264.2, 126.9)
- added P7: CONN_01X03, Pin_Headers:Pin_Header_Straight_1x03_Pitch2.54mm, B.Cu at (266.7, 202.9)
- added P7: CONN_01X03, Pin_Headers:Pin_Header_Straight_1x03_Pitch2.54mm, B.Cu at (266.7, 164.9)
- added P7: CONN_01X03, Pin_Headers:Pin_Header_Straight_1x03_Pitch2.54mm, B.Cu at (266.7, 126.9)
- added Q1: MMBT3904, MyModules:SOT23-132-JRL, B.Cu at (106.8, 181.0)
- added Q1: MMBT3904, MyModules:SOT23-132-JRL, B.Cu at (106.8, 143.0)
- added Q1: MMBT3904, MyModules:SOT23-132-JRL, B.Cu at (106.8, 105.0)
- added Q10: MMBT3904, MyModules:SOT23-132-JRL, B.Cu at (178.8, 193.8)
- added Q10: MMBT3904, MyModules:SOT23-132-JRL, B.Cu at (178.8, 155.8)
- added Q10: MMBT3904, MyModules:SOT23-132-JRL, B.Cu at (178.8, 117.8)
- added Q11: MMBT3904, MyModules:SOT23-132-JRL, B.Cu at (196.8, 180.8)
- added Q11: MMBT3904, MyModules:SOT23-132-JRL, B.Cu at (196.8, 142.8)
- added Q11: MMBT3904, MyModules:SOT23-132-JRL, B.Cu at (196.8, 104.8)
- added Q12: MMBT3904, MyModules:SOT23-132-JRL, B.Cu at (196.8, 193.8)
- added Q12: MMBT3904, MyModules:SOT23-132-JRL, B.Cu at (196.8, 155.8)
- added Q12: MMBT3904, MyModules:SOT23-132-JRL, B.Cu at (196.8, 117.8)
- added Q14: C945, TO_SOT_Packages_SMD:SOT-23, B.Cu at (273.0, 175.9)
- added Q14: C945, TO_SOT_Packages_SMD:SOT-23, B.Cu at (273.0, 137.9)
- added Q14: C945, TO_SOT_Packages_SMD:SOT-23, B.Cu at (273.0, 100.0)
- added Q15: A733, TO_SOT_Packages_SMD:SOT-23, B.Cu at (276.0, 179.9)
- added Q15: A733, TO_SOT_Packages_SMD:SOT-23, B.Cu at (276.0, 141.9)
- added Q15: A733, TO_SOT_Packages_SMD:SOT-23, B.Cu at (276.0, 104.0)
- added Q2: MMBT3904, MyModules:SOT23-132-JRL, B.Cu at (106.8, 193.8)
- added Q2: MMBT3904, MyModules:SOT23-132-JRL, B.Cu at (106.8, 155.8)
- added Q2: MMBT3904, MyModules:SOT23-132-JRL, B.Cu at (106.8, 117.8)
- added Q3: MMBT3904, MyModules:SOT23-132-JRL, B.Cu at (124.8, 181.0)
- added Q3: MMBT3904, MyModules:SOT23-132-JRL, B.Cu at (124.8, 143.0)
- added Q3: MMBT3904, MyModules:SOT23-132-JRL, B.Cu at (124.8, 105.0)
- added Q4: MMBT3904, MyModules:SOT23-132-JRL, B.Cu at (124.8, 193.8)
- added Q4: MMBT3904, MyModules:SOT23-132-JRL, B.Cu at (124.8, 155.8)
- added Q4: MMBT3904, MyModules:SOT23-132-JRL, B.Cu at (124.8, 117.8)
- added Q5: MMBT3904, MyModules:SOT23-132-JRL, B.Cu at (142.8, 180.8)
- added Q5: MMBT3904, MyModules:SOT23-132-JRL, B.Cu at (142.8, 142.8)
- added Q5: MMBT3904, MyModules:SOT23-132-JRL, B.Cu at (142.8, 104.8)
- added Q6: MMBT3904, MyModules:SOT23-132-JRL, B.Cu at (142.8, 193.8)
- added Q6: MMBT3904, MyModules:SOT23-132-JRL, B.Cu at (142.8, 155.8)
- added Q6: MMBT3904, MyModules:SOT23-132-JRL, B.Cu at (142.8, 117.8)
- added Q7: MMBT3904, MyModules:SOT23-132-JRL, B.Cu at (160.8, 181.0)
- added Q7: MMBT3904, MyModules:SOT23-132-JRL, B.Cu at (160.8, 143.0)
- added Q7: MMBT3904, MyModules:SOT23-132-JRL, B.Cu at (160.8, 105.0)
- added Q8: MMBT3904, MyModules:SOT23-132-JRL, B.Cu at (160.8, 193.8)
- added Q8: MMBT3904, MyModules:SOT23-132-JRL, B.Cu at (160.8, 155.8)
- added Q8: MMBT3904, MyModules:SOT23-132-JRL, B.Cu at (160.8, 117.8)
- added Q9: MMBT3904, MyModules:SOT23-132-JRL, B.Cu at (178.8, 180.8)
- added Q9: MMBT3904, MyModules:SOT23-132-JRL, B.Cu at (178.8, 142.8)
- added Q9: MMBT3904, MyModules:SOT23-132-JRL, B.Cu at (178.8, 104.8)
- added R1: 220, MyModules:SM0603-R-YAGEO, B.Cu at (78.8, 198.2)
- added R1: 220, MyModules:SM0603-R-YAGEO, B.Cu at (78.8, 160.2)
- added R1: 220, MyModules:SM0603-R-YAGEO, B.Cu at (78.8, 122.2)
- added R10: 100K, MyModules:SM0603-R-YAGEO, B.Cu at (106.8, 176.5)
- added R10: 100K, MyModules:SM0603-R-YAGEO, B.Cu at (106.8, 138.5)
- added R10: 100K, MyModules:SM0603-R-YAGEO, B.Cu at (106.8, 100.5)
- added R11: 100K, MyModules:SM0603-R-YAGEO, B.Cu at (106.8, 189.2)
- added R11: 100K, MyModules:SM0603-R-YAGEO, B.Cu at (106.8, 151.2)
- added R11: 100K, MyModules:SM0603-R-YAGEO, B.Cu at (106.8, 113.2)
- added R12: 100K, MyModules:SM0603-R-YAGEO, B.Cu at (124.8, 176.5)
- added R12: 100K, MyModules:SM0603-R-YAGEO, B.Cu at (124.8, 138.5)
- added R12: 100K, MyModules:SM0603-R-YAGEO, B.Cu at (124.8, 100.5)
- added R13: 100K, MyModules:SM0603-R-YAGEO, B.Cu at (124.8, 189.2)
- added R13: 100K, MyModules:SM0603-R-YAGEO, B.Cu at (124.8, 151.2)
- added R13: 100K, MyModules:SM0603-R-YAGEO, B.Cu at (124.8, 113.2)
- added R14: 10K, MyModules:SM0603-R-YAGEO, B.Cu at (104.2, 181.5)
- added R14: 10K, MyModules:SM0603-R-YAGEO, B.Cu at (104.2, 143.5)
- added R14: 10K, MyModules:SM0603-R-YAGEO, B.Cu at (104.2, 105.5)
- added R15: 10K, MyModules:SM0603-R-YAGEO, B.Cu at (104.2, 194.2)
- added R15: 10K, MyModules:SM0603-R-YAGEO, B.Cu at (104.2, 156.2)
- added R15: 10K, MyModules:SM0603-R-YAGEO, B.Cu at (104.2, 118.2)
- added R16: 10K, MyModules:SM0603-R-YAGEO, B.Cu at (122.2, 181.5)
- added R16: 10K, MyModules:SM0603-R-YAGEO, B.Cu at (122.2, 143.5)
- added R16: 10K, MyModules:SM0603-R-YAGEO, B.Cu at (122.2, 105.5)
- added R17: 10K, MyModules:SM0603-R-YAGEO, B.Cu at (122.2, 194.2)
- added R17: 10K, MyModules:SM0603-R-YAGEO, B.Cu at (122.2, 156.2)
- added R17: 10K, MyModules:SM0603-R-YAGEO, B.Cu at (122.2, 118.2)
- added R18: 100K, MyModules:SM0603-R-YAGEO, B.Cu at (142.8, 177.8)
- added R18: 100K, MyModules:SM0603-R-YAGEO, B.Cu at (142.8, 139.8)
- added R18: 100K, MyModules:SM0603-R-YAGEO, B.Cu at (142.8, 101.8)
- added R19: 100K, MyModules:SM0603-R-YAGEO, B.Cu at (142.8, 190.8)
- added R19: 100K, MyModules:SM0603-R-YAGEO, B.Cu at (142.8, 152.8)
- added R19: 100K, MyModules:SM0603-R-YAGEO, B.Cu at (142.8, 114.8)
- added R2: 22, MyModules:SM0603-R-YAGEO, B.Cu at (67.0, 194.5)
- added R2: 22, MyModules:SM0603-R-YAGEO, B.Cu at (67.0, 156.5)
- added R2: 22, MyModules:SM0603-R-YAGEO, B.Cu at (67.0, 118.5)
- added R20: 100K, MyModules:SM0603-R-YAGEO, B.Cu at (160.8, 177.8)
- added R20: 100K, MyModules:SM0603-R-YAGEO, B.Cu at (160.8, 139.8)
- added R20: 100K, MyModules:SM0603-R-YAGEO, B.Cu at (160.8, 101.8)
- added R21: 100K, MyModules:SM0603-R-YAGEO, B.Cu at (160.8, 190.8)
- added R21: 100K, MyModules:SM0603-R-YAGEO, B.Cu at (160.8, 152.8)
- added R21: 100K, MyModules:SM0603-R-YAGEO, B.Cu at (160.8, 114.8)
- added R22: 100K, MyModules:SM0603-R-YAGEO, B.Cu at (142.8, 176.2)
- added R22: 100K, MyModules:SM0603-R-YAGEO, B.Cu at (142.8, 138.2)
- added R22: 100K, MyModules:SM0603-R-YAGEO, B.Cu at (142.8, 100.2)
- added R23: 100K, MyModules:SM0603-R-YAGEO, B.Cu at (142.8, 189.2)
- added R23: 100K, MyModules:SM0603-R-YAGEO, B.Cu at (142.8, 151.2)
- added R23: 100K, MyModules:SM0603-R-YAGEO, B.Cu at (142.8, 113.2)
- added R24: 100K, MyModules:SM0603-R-YAGEO, B.Cu at (160.8, 176.2)
- added R24: 100K, MyModules:SM0603-R-YAGEO, B.Cu at (160.8, 138.2)
- added R24: 100K, MyModules:SM0603-R-YAGEO, B.Cu at (160.8, 100.2)
- added R25: 100K, MyModules:SM0603-R-YAGEO, B.Cu at (160.8, 189.2)
- added R25: 100K, MyModules:SM0603-R-YAGEO, B.Cu at (160.8, 151.2)
- added R25: 100K, MyModules:SM0603-R-YAGEO, B.Cu at (160.8, 113.2)
- added R26: 10K, MyModules:SM0603-R-YAGEO, B.Cu at (140.2, 181.5)
- added R26: 10K, MyModules:SM0603-R-YAGEO, B.Cu at (140.2, 143.5)
- added R26: 10K, MyModules:SM0603-R-YAGEO, B.Cu at (140.2, 105.5)
- added R27: 10K, MyModules:SM0603-R-YAGEO, B.Cu at (140.2, 194.2)
- added R27: 10K, MyModules:SM0603-R-YAGEO, B.Cu at (140.2, 156.2)
- added R27: 10K, MyModules:SM0603-R-YAGEO, B.Cu at (140.2, 118.2)
- added R28: 10K, MyModules:SM0603-R-YAGEO, B.Cu at (158.2, 181.5)
- added R28: 10K, MyModules:SM0603-R-YAGEO, B.Cu at (158.2, 143.5)
- added R28: 10K, MyModules:SM0603-R-YAGEO, B.Cu at (158.2, 105.5)
- added R29: 10K, MyModules:SM0603-R-YAGEO, B.Cu at (158.2, 194.2)
- added R29: 10K, MyModules:SM0603-R-YAGEO, B.Cu at (158.2, 156.2)
- added R29: 10K, MyModules:SM0603-R-YAGEO, B.Cu at (158.2, 118.2)
- added R3: 220, MyModules:SM0603-R-YAGEO, B.Cu at (48.0, 148.5)
- added R3: 220, MyModules:SM0603-R-YAGEO, B.Cu at (48.0, 186.5)
- added R3: 220, MyModules:SM0603-R-YAGEO, B.Cu at (48.0, 110.5)
- added R30: 100K, MyModules:SM0603-R-YAGEO, B.Cu at (178.8, 177.8)
- added R30: 100K, MyModules:SM0603-R-YAGEO, B.Cu at (178.8, 139.8)
- added R30: 100K, MyModules:SM0603-R-YAGEO, B.Cu at (178.8, 101.8)
- added R31: 100K, MyModules:SM0603-R-YAGEO, B.Cu at (178.8, 190.8)
- added R31: 100K, MyModules:SM0603-R-YAGEO, B.Cu at (178.8, 152.8)
- added R31: 100K, MyModules:SM0603-R-YAGEO, B.Cu at (178.8, 114.8)
- added R32: 100K, MyModules:SM0603-R-YAGEO, B.Cu at (196.8, 177.8)
- added R32: 100K, MyModules:SM0603-R-YAGEO, B.Cu at (196.8, 139.8)
- added R32: 100K, MyModules:SM0603-R-YAGEO, B.Cu at (196.8, 101.8)
- added R33: 100K, MyModules:SM0603-R-YAGEO, B.Cu at (196.8, 190.8)
- added R33: 100K, MyModules:SM0603-R-YAGEO, B.Cu at (196.8, 152.8)
- added R33: 100K, MyModules:SM0603-R-YAGEO, B.Cu at (196.8, 114.8)
- added R34: 100K, MyModules:SM0603-R-YAGEO, B.Cu at (178.8, 176.2)
- added R34: 100K, MyModules:SM0603-R-YAGEO, B.Cu at (178.8, 138.2)
- added R34: 100K, MyModules:SM0603-R-YAGEO, B.Cu at (178.8, 100.2)
- added R35: 100K, MyModules:SM0603-R-YAGEO, B.Cu at (178.8, 189.2)
- added R35: 100K, MyModules:SM0603-R-YAGEO, B.Cu at (178.8, 151.2)
- added R35: 100K, MyModules:SM0603-R-YAGEO, B.Cu at (178.8, 113.2)
- added R36: 100K, MyModules:SM0603-R-YAGEO, B.Cu at (196.8, 176.2)
- added R36: 100K, MyModules:SM0603-R-YAGEO, B.Cu at (196.8, 138.2)
- added R36: 100K, MyModules:SM0603-R-YAGEO, B.Cu at (196.8, 100.2)
- added R37: 100K, MyModules:SM0603-R-YAGEO, B.Cu at (196.8, 189.2)
- added R37: 100K, MyModules:SM0603-R-YAGEO, B.Cu at (196.8, 151.2)
- added R37: 100K, MyModules:SM0603-R-YAGEO, B.Cu at (196.8, 113.2)
- added R38: 10K, MyModules:SM0603-R-YAGEO, B.Cu at (176.2, 181.5)
- added R38: 10K, MyModules:SM0603-R-YAGEO, B.Cu at (176.2, 143.5)
- added R38: 10K, MyModules:SM0603-R-YAGEO, B.Cu at (176.2, 105.5)
- added R39: 10K, MyModules:SM0603-R-YAGEO, B.Cu at (176.2, 194.2)
- added R39: 10K, MyModules:SM0603-R-YAGEO, B.Cu at (176.2, 156.2)
- added R39: 10K, MyModules:SM0603-R-YAGEO, B.Cu at (176.2, 118.2)
- added R4: 1K, MyModules:SM0603-R-YAGEO, B.Cu at (88.5, 178.5)
- added R4: 1K, MyModules:SM0603-R-YAGEO, B.Cu at (88.5, 140.5)
- added R4: 1K, MyModules:SM0603-R-YAGEO, B.Cu at (88.5, 102.5)
- added R40: 10K, MyModules:SM0603-R-YAGEO, B.Cu at (194.2, 181.5)
- added R40: 10K, MyModules:SM0603-R-YAGEO, B.Cu at (194.2, 143.5)
- added R40: 10K, MyModules:SM0603-R-YAGEO, B.Cu at (194.2, 105.5)
- added R41: 10K, MyModules:SM0603-R-YAGEO, B.Cu at (194.2, 194.2)
- added R41: 10K, MyModules:SM0603-R-YAGEO, B.Cu at (194.2, 156.2)
- added R41: 10K, MyModules:SM0603-R-YAGEO, B.Cu at (194.2, 118.2)
- added R42: 47K, MyModules:SM0603-R-YAGEO, B.Cu at (88.5, 182.0)
- added R42: 47K, MyModules:SM0603-R-YAGEO, B.Cu at (88.5, 144.0)
- added R42: 47K, MyModules:SM0603-R-YAGEO, B.Cu at (88.5, 106.0)
- added R43: 100K, MyModules:SM0603-R-YAGEO, B.Cu at (87.0, 191.8)
- added R43: 100K, MyModules:SM0603-R-YAGEO, B.Cu at (87.0, 153.8)
- added R43: 100K, MyModules:SM0603-R-YAGEO, B.Cu at (87.0, 115.8)
- added R44: 47K, MyModules:SM0603-R-YAGEO, B.Cu at (142.4, 200.5)
- added R44: 47K, MyModules:SM0603-R-YAGEO, B.Cu at (142.4, 162.5)
- added R44: 47K, MyModules:SM0603-R-YAGEO, B.Cu at (142.4, 124.5)
- added R45: 47K, MyModules:SM0603-R-YAGEO, B.Cu at (151.8, 201.5)
- added R45: 47K, MyModules:SM0603-R-YAGEO, B.Cu at (151.8, 163.5)
- added R45: 47K, MyModules:SM0603-R-YAGEO, B.Cu at (151.8, 125.5)
- added R46: 33K, MyModules:SM0603-R-YAGEO, B.Cu at (222.0, 202.0)
- added R46: 33K, MyModules:SM0603-R-YAGEO, B.Cu at (222.0, 164.0)
- added R46: 33K, MyModules:SM0603-R-YAGEO, B.Cu at (222.0, 126.0)
- added R47: 33K, MyModules:SM0603-R-YAGEO, B.Cu at (222.0, 203.2)
- added R47: 33K, MyModules:SM0603-R-YAGEO, B.Cu at (222.0, 165.2)
- added R47: 33K, MyModules:SM0603-R-YAGEO, B.Cu at (222.0, 127.2)
- added R48: 33K, MyModules:SM0603-R-YAGEO, B.Cu at (224.5, 200.0)
- added R48: 33K, MyModules:SM0603-R-YAGEO, B.Cu at (224.5, 162.0)
- added R48: 33K, MyModules:SM0603-R-YAGEO, B.Cu at (224.5, 124.0)
- added R49: 33K, MyModules:SM0603-R-YAGEO, B.Cu at (227.8, 200.0)
- added R49: 33K, MyModules:SM0603-R-YAGEO, B.Cu at (227.8, 162.0)
- added R49: 33K, MyModules:SM0603-R-YAGEO, B.Cu at (227.8, 124.0)
- added R5: 1K, MyModules:SM0603-R-YAGEO, B.Cu at (88.5, 191.8)
- added R5: 1K, MyModules:SM0603-R-YAGEO, B.Cu at (88.5, 153.8)
- added R5: 1K, MyModules:SM0603-R-YAGEO, B.Cu at (88.5, 115.8)
- added R50: 33K, MyModules:SM0603-R-YAGEO, B.Cu at (231.5, 206.2)
- added R50: 33K, MyModules:SM0603-R-YAGEO, B.Cu at (231.5, 168.2)
- added R50: 33K, MyModules:SM0603-R-YAGEO, B.Cu at (231.5, 130.2)
- added R51: 22K, MyModules:SM0603-R-YAGEO, B.Cu at (238.5, 165.2)
- added R51: 22K, MyModules:SM0603-R-YAGEO, B.Cu at (238.5, 203.2)
- added R51: 22K, MyModules:SM0603-R-YAGEO, B.Cu at (238.5, 127.2)
- added R52: 33K, MyModules:SM0603-R-YAGEO, B.Cu at (234.8, 162.8)
- added R52: 33K, MyModules:SM0603-R-YAGEO, B.Cu at (234.8, 200.8)
- added R52: 33K, MyModules:SM0603-R-YAGEO, B.Cu at (234.8, 124.8)
- added R54: 27K, MyModules:SM0603-R-YAGEO, B.Cu at (251.8, 185.0)
- added R54: 27K, MyModules:SM0603-R-YAGEO, B.Cu at (251.8, 147.0)
- added R54: 27K, MyModules:SM0603-R-YAGEO, B.Cu at (251.8, 109.0)
- added R55: 3.3K, MyModules:SM0603-R-YAGEO, B.Cu at (251.8, 188.2)
- added R55: 3.3K, MyModules:SM0603-R-YAGEO, B.Cu at (251.8, 150.2)
- added R55: 3.3K, MyModules:SM0603-R-YAGEO, B.Cu at (251.8, 112.2)
- added R56: 1K, MyModules:SM0603-R-YAGEO, B.Cu at (254.0, 181.8)
- added R56: 1K, MyModules:SM0603-R-YAGEO, B.Cu at (254.0, 143.8)
- added R56: 1K, MyModules:SM0603-R-YAGEO, B.Cu at (254.0, 105.8)
- added R57: 68R, MyModules:SM0603-R-YAGEO, B.Cu at (270.7, 197.2)
- added R57: 68R, MyModules:SM0603-R-YAGEO, B.Cu at (270.7, 159.2)
- added R57: 68R, MyModules:SM0603-R-YAGEO, B.Cu at (270.7, 121.2)
- added R58: 22K, MyModules:SM0603-R-YAGEO, B.Cu at (270.2, 176.2)
- added R58: 22K, MyModules:SM0603-R-YAGEO, B.Cu at (270.2, 138.2)
- added R58: 22K, MyModules:SM0603-R-YAGEO, B.Cu at (270.2, 100.2)
- added R59: 22K, MyModules:SM0603-R-YAGEO, B.Cu at (275.9, 177.4)
- added R59: 22K, MyModules:SM0603-R-YAGEO, B.Cu at (275.9, 139.4)
- added R59: 22K, MyModules:SM0603-R-YAGEO, B.Cu at (275.9, 101.4)
- added R6: 100K, MyModules:SM0603-R-YAGEO, B.Cu at (106.8, 178.0)
- added R6: 100K, MyModules:SM0603-R-YAGEO, B.Cu at (106.8, 140.0)
- added R6: 100K, MyModules:SM0603-R-YAGEO, B.Cu at (106.8, 102.0)
- added R60: 68R, MyModules:SM0603-R-YAGEO, B.Cu at (276.2, 202.8)
- added R60: 68R, MyModules:SM0603-R-YAGEO, B.Cu at (276.2, 164.8)
- added R60: 68R, MyModules:SM0603-R-YAGEO, B.Cu at (276.2, 126.8)
- added R61: 180, Resistors_SMD:R_0805, B.Cu at (276.0, 174.9)
- added R61: 180, Resistors_SMD:R_0805, B.Cu at (276.0, 136.9)
- added R61: 180, Resistors_SMD:R_0805, B.Cu at (276.0, 99.0)
- added R62: 180, Resistors_SMD:R_0805, B.Cu at (271.8, 146.2)
- added R62: 180, Resistors_SMD:R_0805, B.Cu at (271.8, 184.2)
- added R62: 180, Resistors_SMD:R_0805, B.Cu at (271.8, 108.2)
- added R63: 22R, Resistors_SMD:R_0805, B.Cu at (266.3, 148.1)
- added R63: 22R, Resistors_SMD:R_0805, B.Cu at (266.3, 186.1)
- added R63: 22R, Resistors_SMD:R_0805, B.Cu at (266.3, 110.1)
- added R64: 22R, Resistors_SMD:R_0805, B.Cu at (268.2, 148.1)
- added R64: 22R, Resistors_SMD:R_0805, B.Cu at (268.2, 186.1)
- added R64: 22R, Resistors_SMD:R_0805, B.Cu at (268.2, 110.1)
- added R67: 120, Resistors_SMD:R_0805, B.Cu at (259.1, 199.9)
- added R67: 120, Resistors_SMD:R_0805, B.Cu at (259.1, 161.9)
- added R67: 120, Resistors_SMD:R_0805, B.Cu at (259.1, 123.9)
- added R7: 100K, MyModules:SM0603-R-YAGEO, B.Cu at (106.8, 190.8)
- added R7: 100K, MyModules:SM0603-R-YAGEO, B.Cu at (106.8, 152.8)
- added R7: 100K, MyModules:SM0603-R-YAGEO, B.Cu at (106.8, 114.8)
- added R8: 100K, MyModules:SM0603-R-YAGEO, B.Cu at (124.8, 178.0)
- added R8: 100K, MyModules:SM0603-R-YAGEO, B.Cu at (124.8, 140.0)
- added R8: 100K, MyModules:SM0603-R-YAGEO, B.Cu at (124.8, 102.0)
- added R9: 100K, MyModules:SM0603-R-YAGEO, B.Cu at (124.8, 190.8)
- added R9: 100K, MyModules:SM0603-R-YAGEO, B.Cu at (124.8, 152.8)
- added R9: 100K, MyModules:SM0603-R-YAGEO, B.Cu at (124.8, 114.8)
- added REF**: fiducial-1mm, MyModules:fiducial-1mm, B.Cu at (283.5, 212.5)
- added REF**: fiducial-1mm, MyModules:fiducial-1mm, B.Cu at (20.0, 54.5)
- added REF**: fiducial-1mm, MyModules:fiducial-1mm, B.Cu at (289.0, 207.0)
- added REF**: fiducial-1mm, MyModules:fiducial-1mm, B.Cu at (289.0, 169.0)
- added REF**: fiducial-1mm, MyModules:fiducial-1mm, B.Cu at (14.5, 174.0)
- added REF**: fiducial-1mm, MyModules:fiducial-1mm, B.Cu at (14.5, 136.0)
- added REF**: fiducial-1mm, MyModules:fiducial-1mm, B.Cu at (14.5, 98.0)
- added REF**: fiducial-1mm, MyModules:fiducial-1mm, B.Cu at (289.0, 131.0)
- added REF***: WEEE-Logo_5.6x8mm_SilkScreen, Symbols:WEEE-Logo_5.6x8mm_SilkScreen, F.Cu at (186.0, 204.5)
- added REF***: WEEE-Logo_5.6x8mm_SilkScreen, Symbols:WEEE-Logo_5.6x8mm_SilkScreen, F.Cu at (186.0, 166.5)
- added REF***: WEEE-Logo_5.6x8mm_SilkScreen, Symbols:WEEE-Logo_5.6x8mm_SilkScreen, F.Cu at (186.0, 128.5)
- added REF***: WEEE-Logo_5.6x8mm_SilkScreen, Symbols:WEEE-Logo_5.6x8mm_SilkScreen, F.Cu at (186.0, 90.5)
- added TP2: CONN_1, MyModules:TEST_POINT_LOOP_4592, B.Cu at (213.8, 160.0)
- added TP2: CONN_1, MyModules:TEST_POINT_LOOP_4592, B.Cu at (213.8, 198.0)
- added TP2: CONN_1, MyModules:TEST_POINT_LOOP_4592, B.Cu at (213.8, 122.0)
- added U1: 74HC165, Housings_SSOP:TSSOP-16_4.4x5mm_Pitch0.65mm, B.Cu at (103.5, 204.0)
- added U1: 74HC165, Housings_SSOP:TSSOP-16_4.4x5mm_Pitch0.65mm, B.Cu at (103.5, 166.0)
- added U1: 74HC165, Housings_SSOP:TSSOP-16_4.4x5mm_Pitch0.65mm, B.Cu at (103.5, 128.0)
- added U2: 74HC165, Housings_SSOP:TSSOP-16_4.4x5mm_Pitch0.65mm, B.Cu at (134.5, 204.0)
- added U2: 74HC165, Housings_SSOP:TSSOP-16_4.4x5mm_Pitch0.65mm, B.Cu at (134.5, 166.0)
- added U2: 74HC165, Housings_SSOP:TSSOP-16_4.4x5mm_Pitch0.65mm, B.Cu at (134.5, 128.0)
- added U3: VX078-500, MyModules:CUI_VXO780XX-500, B.Cu at (14.5, 203.0)
- added U3: VX078-500, MyModules:CUI_VXO780XX-500, B.Cu at (14.5, 165.0)
- added U3: VX078-500, MyModules:CUI_VXO780XX-500, B.Cu at (14.5, 127.0)
- added U4: VX078-500, MyModules:CUI_VXO780XX-500, B.Cu at (62.5, 203.0)
- added U4: VX078-500, MyModules:CUI_VXO780XX-500, B.Cu at (62.5, 165.0)
- added U4: VX078-500, MyModules:CUI_VXO780XX-500, B.Cu at (62.5, 127.0)
- added U5: 4558, Housings_SSOP:TSSOP-8_4.4x3mm_Pitch0.65mm, B.Cu at (233.0, 203.5)
- added U5: 4558, Housings_SSOP:TSSOP-8_4.4x3mm_Pitch0.65mm, B.Cu at (233.0, 165.5)
- added U5: 4558, Housings_SSOP:TSSOP-8_4.4x3mm_Pitch0.65mm, B.Cu at (233.0, 127.5)
- added U6: 4558, Housings_SSOP:TSSOP-8_4.4x3mm_Pitch0.65mm, B.Cu at (267.2, 178.4)
- added U6: 4558, Housings_SSOP:TSSOP-8_4.4x3mm_Pitch0.65mm, B.Cu at (267.2, 140.4)
- added U6: 4558, Housings_SSOP:TSSOP-8_4.4x3mm_Pitch0.65mm, B.Cu at (267.2, 102.5)
- added U7: 74HC1G125, Housings_SSOP:TSOP-5_1.65x3.05mm_Pitch0.95mm, B.Cu at (145.5, 200.5)
- added U7: 74HC1G125, Housings_SSOP:TSOP-5_1.65x3.05mm_Pitch0.95mm, B.Cu at (145.5, 162.5)
- added U7: 74HC1G125, Housings_SSOP:TSOP-5_1.65x3.05mm_Pitch0.95mm, B.Cu at (145.5, 124.5)
- added X1: MIDI OUT, MyModules:SD-50BV-5DIN-SLOTS, F.Cu at (39.0, 186.2)
- added X1: MIDI OUT, MyModules:SD-50BV-5DIN-SLOTS, F.Cu at (39.0, 148.2)
- added X1: MIDI OUT, MyModules:SD-50BV-5DIN-SLOTS, F.Cu at (39.0, 110.2)
- added X2: SYNC24, MyModules:SD-50BV-5DIN-SLOTS, F.Cu at (61.0, 186.2)
- added X2: SYNC24, MyModules:SD-50BV-5DIN-SLOTS, F.Cu at (61.0, 148.2)
- added X2: SYNC24, MyModules:SD-50BV-5DIN-SLOTS, F.Cu at (61.0, 110.2)
Routing:
- net +5V: track 337.9 -> 1351.5 mm, vias 17 -> 68
- net +V: track 309.1 -> 1236.5 mm, vias 4 -> 16
- net -V: track 279.0 -> 1116.0 mm, vias 5 -> 20
- net GNDD: track 113.6 -> 454.3 mm, vias 8 -> 32
- net DIN_RUN_STOP: track 102.3 -> 409.3 mm, vias 1 -> 4
- net /OH: track 68.9 -> 275.8 mm
- net /CP: track 64.8 -> 259.4 mm
- net /CH: track 63.4 -> 253.7 mm
- net Net-(C16-Pad1): track 61.7 -> 247.0 mm
- net /MA: track 58.4 -> 233.7 mm
- net DIN_TEMPO_CLK: track 58.4 -> 233.4 mm
- net /CB: track 54.9 -> 219.7 mm
- net GND: track 54.7 -> 218.6 mm, vias 13 -> 52
- net /HT: track 49.0 -> 195.9 mm
- net Net-(R1-Pad1): track 46.2 -> 185.0 mm
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Other:
- board size 279.5 x 38 mm -> 279.5 x 164 mm
- board text added: "System80 Inc. Toronto, Ontario, Canada"
- board text added: "V-CUT"
