File: 880_enclosure_subboards.kicad_pcb (KiCad board)
At the start: 2 copper layers, 54.3 x 38 mm, 16 parts, among them J23 JACK_STEREO, J24 JACK_TRS_SWITCHED, J25 JACK_STEREO, P10 CONN_01X02, P11 CONN_01X03, P6 CONN_01X04, P8 CONN_01X03, SW1 SPST

Commit message: v1.1 ordered plus sub boards
Other:
- board text added: "880ENC 6/2019"
Changed lines of the file:
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@@
     (area 296.949999 57.449999 351.304027 95.550933)
     (thickness 1.6)
-    (drawings 41)
+    (drawings 42)
     (tracks 51)
     (zones 0)
@@
     )
   )
+  (gr_text "880ENC 6/2019" (at 303.5 94.25 360) (layer B.SilkS)
+    (effects (font (size 1 1) (thickness 0.15)) (justify mirror))
+  )
   (gr_line (start 334.25 86.75) (end 334.25 77.75) (layer Edge.Cuts) (width 0.1))

Commit message: first update in a long while. this version and gone through production
Other:
- board text added: "880ENC 2/2020"
- board text removed: "880ENC 6/2019"
Changed lines of the file:
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@@
     (mod_text_size 1 1)
     (mod_text_width 0.15)
-    (pad_size 1 1)
-    (pad_drill 1)
+    (pad_size 1.65 4.5)
+    (pad_drill 0.6)
     (pad_to_mask_clearance 0.05)
     (aux_axis_origin 0 0)
@@
       (effects (font (size 1 1) (thickness 0.15)))
     )
-    (pad 2 thru_hole rect (at 0 0 180) (size 1.5 4.5) (drill oval 0.6 3.8) (layers *.Cu *.Mask F.SilkS)
+    (pad 2 thru_hole rect (at 0 0 180) (size 1.65 4.5) (drill oval 0.6 3.8) (layers *.Cu *.Mask F.SilkS)
       (net 8 "Net-(P10-Pad1)"))
-    (pad 1 thru_hole rect (at -4.5 0 180) (size 1.5 4.5) (drill oval 0.6 3.8) (layers *.Cu *.Mask F.SilkS)
+    (pad 1 thru_hole rect (at -4.5 0 180) (size 1.65 4.5) (drill oval 0.6 3.8) (layers *.Cu *.Mask F.SilkS)
       (net 9 "Net-(P10-Pad2)"))
   )
@@
       (effects (font (size 1 1) (thickness 0.15)))
     )
-    (pad 1 thru_hole rect (at 0 0 90) (size 2.6 1.8) (drill 1.2) (layers *.Cu *.Mask)
+    (pad 1 thru_hole rect (at 0 0 90) (size 2.75 2) (drill 1.45 (offset -0.15 -0.1)) (layers *.Cu *.Mask)
       (net 8 "Net-(P10-Pad1)"))
-    (pad 2 thru_hole oval (at 0 2.54 90) (size 2.6 1.8) (drill 1.2) (layers *.Cu *.Mask)
+    (pad 2 thru_hole oval (at 0 2.54 90) (size 2.75 2) (drill 1.45 (offset -0.15 0.1)) (layers *.Cu *.Mask)
       (net 9 "Net-(P10-Pad2)"))
     (model ${KISYS3DMOD}/Pin_Headers.3dshapes/Pin_Header_Straight_1x02_Pitch2.54mm.wrl
@@
     )
   )
-  (gr_text "880ENC 6/2019" (at 303.5 94.25 360) (layer B.SilkS)
+  (gr_text "880ENC 2/2020" (at 303.5 94.25) (layer B.SilkS)
     (effects (font (size 1 1) (thickness 0.15)) (justify mirror))
   )
