File: 880_enclosure_unit.kicad_pcb (KiCad board)
At the start: 4 copper layers, 279.5 x 38 mm, 164 parts, among them CON1 BARREL_JACK, J1 RUN/STOP, J10 RS IN, J11 CP IN, J12 MA IN, J13 CB IN, J14 CY IN, J15 OH IN, J16 CH IN, J17 IN 1, J18 IN 2, J19 IN 3, J2 SYNC24 CLK, J20 IN 4, J21 MULT IN, J22 SUM, J3 ASSIGN 1, J4 ASSIGN 2, J5 BD IN, J6 SD IN, J7 LT IN, J8 MT IN, J9 HT IN, P1 CONN_02X03, P2 CONN_01X02, P3 CONN_02X08, P4 CONN_01X03, P5 CONN_01X04, P7 CONN_01X03, Q1 MMBT3904, Q10 MMBT3904, Q11 MMBT3904, Q12 MMBT3904, Q14 C945, Q15 A733, Q2 MMBT3904, Q3 MMBT3904, Q4 MMBT3904, Q5 MMBT3904, Q6 MMBT3904, Q7 MMBT3904, Q8 MMBT3904, Q9 MMBT3904, U1 74HC165, U2 74HC165, U3 VX078-500, U4 VX078-500, U5 4558, U6 4558, U7 74HC1G125, X1 MIDI OUT, X2 SYNC24

Commit message: getting ready to panelize for production
Parts:
- added G***: LOGO, LOGO, F.Cu at (151.0, 92.0)
- added REF**: fiducial-1mm, MyModules:fiducial-1mm, B.Cu at (289.0, 93.0)
- added REF**: fiducial-1mm, MyModules:fiducial-1mm, B.Cu at (14.5, 60.0)
Other:
- board text added: "System80 Inc. Toronto, Ontario, Canada"

Commit message: first update in a long while. this version and gone through production
Changed lines of the file:
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@@
 (kicad_pcb (version 4) (host pcbnew 4.0.2-stable)
   (general
-    (links 0)
+    (links 356)
     (no_connects 0)
     (area 11.944431 57.449999 291.550001 95.551147)
@@
     (add_net GND)
   )
+  (module Housings_SSOP:TSOP-5_1.65x3.05mm_Pitch0.95mm (layer B.Cu)
+    (at 145.5 86.5 180)
+    (descr "TSOP-5 package (comparable to TSOT-23), https://www.vishay.com/docs/71200/71200.pdf")
+    (tags "Jedec MO-193C TSOP-5L")
+    (attr smd)
+    (fp_text reference U7 (at 0 2.45 180) (layer B.SilkS)
+      (effects (font (size 1 1) (thickness 0.15)) (justify mirror))
+    )
+    (fp_text value 74HC1G125 (at 0 -2.5 180) (layer B.Fab)
+      (effects (font (size 1 1) (thickness 0.15)) (justify mirror))
+    )
+    (fp_text user %R (at 0 0 450) (layer B.Fab)
+      (effects (font (size 0.5 0.5) (thickness 0.075)) (justify mirror))
+    )
+    (fp_line (start -0.8 -1.6) (end 0.8 -1.6) (layer B.SilkS) (width 0.12))
+    (fp_line (start 0.8 1.6) (end -1.5 1.6) (layer B.SilkS) (width 0.12))
+    (fp_line (start -0.825 1.1) (end -0.425 1.525) (layer B.Fab) (width 0.1))
+    (fp_line (start 0.825 1.525) (end -0.425 1.525) (layer B.Fab) (width 0.1))
+    (fp_line (start -0.825 1.1) (end -0.825 -1.525) (layer B.Fab) (width 0.1))
+    (fp_line (start 0.825 -1.525) (end -0.825 -1.525) (layer B.Fab) (width 0.1))
+    (fp_line (start 0.825 1.525) (end 0.825 -1.525) (layer B.Fab) (width 0.1))
+    (fp_line (start -1.76 1.78) (end 1.76 1.78) (layer B.CrtYd) (width 0.05))
+    (fp_line (start -1.76 1.78) (end -1.76 -1.77) (layer B.CrtYd) (width 0.05))
+    (fp_line (start 1.76 -1.77) (end 1.76 1.78) (layer B.CrtYd) (width 0.05))
+    (fp_line (start 1.76 -1.77) (end -1.76 -1.77) (layer B.CrtYd) (width 0.05))
+    (pad 1 smd rect (at -1.16 0.95 180) (size 0.7 0.51) (layers B.Cu B.Paste B.Mask)
+      (net 38 DIN_RUN_STOP))
+    (pad 2 smd rect (at -1.16 0 180) (size 0.7 0.51) (layers B.Cu B.Paste B.Mask)
+      (net 109 "Net-(U2-Pad9)"))
+    (pad 3 smd rect (at -1.16 -0.95 180) (size 0.7 0.51) (layers B.Cu B.Paste B.Mask)
+      (net 106 GNDD))
+    (pad 4 smd rect (at 1.16 -0.95 180) (size 0.7 0.51) (layers B.Cu B.Paste B.Mask)
+      (net 35 ISP_MISO))
+    (pad 6 smd rect (at 1.16 0.95 180) (size 0.7 0.51) (layers B.Cu B.Paste B.Mask)
+      (net 3 +5V))
+    (model ${KISYS3DMOD}/Housings_SSOP.3dshapes/TSOP-5_1.65x3.05mm_Pitch0.95mm.wrl
+      (at (xyz 0 0 0))
+      (scale (xyz 1 1 1))
+      (rotate (xyz 0 0 0))
+    )
+  )
   (module LOGO (layer F.Cu)
     (at 151 92)
@@
       (solder_mask_margin 0.5) (clearance 0.75))
   )
-  (module Housings_SSOP:TSOP-5_1.65x3.05mm_Pitch0.95mm (layer B.Cu)
-    (at 145.5 86.5 180)
-    (descr "TSOP-5 package (comparable to TSOT-23), https://www.vishay.com/docs/71200/71200.pdf")
-    (tags "Jedec MO-193C TSOP-5L")
-    (attr smd)
-    (fp_text reference U7 (at 0 2.45 180) (layer B.SilkS)
-      (effects (font (size 1 1) (thickness 0.15)) (justify mirror))
-    )
-    (fp_text value 74HC1G125 (at 0 -2.5 180) (layer B.Fab)
-      (effects (font (size 1 1) (thickness 0.15)) (justify mirror))
-    )
-    (fp_text user %R (at 0 0 450) (layer B.Fab)
-      (effects (font (size 0.5 0.5) (thickness 0.075)) (justify mirror))
-    )
-    (fp_line (start -0.8 -1.6) (end 0.8 -1.6) (layer B.SilkS) (width 0.12))
-    (fp_line (start 0.8 1.6) (end -1.5 1.6) (layer B.SilkS) (width 0.12))
-    (fp_line (start -0.825 1.1) (end -0.425 1.525) (layer B.Fab) (width 0.1))
-    (fp_line (start 0.825 1.525) (end -0.425 1.525) (layer B.Fab) (width 0.1))
-    (fp_line (start -0.825 1.1) (end -0.825 -1.525) (layer B.Fab) (width 0.1))
-    (fp_line (start 0.825 -1.525) (end -0.825 -1.525) (layer B.Fab) (width 0.1))
-    (fp_line (start 0.825 1.525) (end 0.825 -1.525) (layer B.Fab) (width 0.1))
-    (fp_line (start -1.76 1.78) (end 1.76 1.78) (layer B.CrtYd) (width 0.05))
-    (fp_line (start -1.76 1.78) (end -1.76 -1.77) (layer B.CrtYd) (width 0.05))
-    (fp_line (start 1.76 -1.77) (end 1.76 1.78) (layer B.CrtYd) (width 0.05))
-    (fp_line (start 1.76 -1.77) (end -1.76 -1.77) (layer B.CrtYd) (width 0.05))
-    (pad 1 smd rect (at -1.16 0.95 180) (size 0.7 0.51) (layers B.Cu B.Paste B.Mask)
-      (net 38 DIN_RUN_STOP))
-    (pad 2 smd rect (at -1.16 0 180) (size 0.7 0.51) (layers B.Cu B.Paste B.Mask)
-      (net 109 "Net-(U2-Pad9)"))
-    (pad 3 smd rect (at -1.16 -0.95 180) (size 0.7 0.51) (layers B.Cu B.Paste B.Mask)
-      (net 106 GNDD))
-    (pad 4 smd rect (at 1.16 -0.95 180) (size 0.7 0.51) (layers B.Cu B.Paste B.Mask)
-      (net 35 ISP_MISO))
-    (pad 6 smd rect (at 1.16 0.95 180) (size 0.7 0.51) (layers B.Cu B.Paste B.Mask)
-      (net 3 +5V))
-    (model ${KISYS3DMOD}/Housings_SSOP.3dshapes/TSOP-5_1.65x3.05mm_Pitch0.95mm.wrl
-      (at (xyz 0 0 0))
-      (scale (xyz 1 1 1))
-      (rotate (xyz 0 0 0))
-    )
-  )
   (module MyModules:SM0603-C-MURATA (layer B.Cu)
     (at 120.5 75.85 90)
@@
     (at 140.9 86.5 270)
     (attr smd)
-    (fp_text reference C20 (at 0 1.4 270) (layer B.SilkS)
+    (fp_text reference C20 (at -2.4 0 270) (layer B.SilkS)
       (effects (font (size 0.6096 0.6096) (thickness 0.1524)) (justify mirror))
     )
@@
     (at 142.4 86.5 270)
     (attr smd)
-    (fp_text reference R44 (at 0 1.4 270) (layer B.SilkS)
+    (fp_text reference R44 (at -2.4 0 270) (layer B.SilkS)
       (effects (font (size 0.6096 0.6096) (thickness 0.1524)) (justify mirror))
     )
@@
   (segment (start 176.25 79.4) (end 175.199996 79.4) (width 0.35) (layer B.Cu) (net 3))
   (via (at 175.199996 79.4) (size 1) (drill 0.5) (layers F.Cu B.Cu) (net 3))
-  (segment (start 87 67.25) (end 87 70.5) (width 0.35) (layer B.Cu) (net 3))
-  (segment (start 87 70.5) (end 88.5 72) (width 0.35) (layer B.Cu) (net 3))
+  (segment (start 87 67.25) (end 87 70.5) (width 0.5) (layer B.Cu) (net 3))
+  (segment (start 87 70.5) (end 88.5 72) (width 0.5) (layer B.Cu) (net 3))
   (segment (start 87 67.25) (end 93.65 67.25) (width 0.5) (layer F.Cu) (net 3))
   (segment (start 93.65 67.25) (end 94.3 66.6) (width 0.5) (layer F.Cu) (net 3))
